File: mastermind_kicad/mastermind.kicad_sch (KiCad schematic)
At the start: 9 parts, among them SW1 Button 1, SW2 Button 2, SW3 Button 3, U1 LED matrix 16x16 (WS2812)

Commit message: Updated Code, Docu, Schematic
Parts:
- removed A1: Arduino UNO R3, symbol MCU_Module:Arduino_UNO_R3
- added A1: Arduino Mega 2560 R3, symbol Custom:Arduino_Mega2560_R3
Connections:
- net +3V3: now also A1.3V3
- net +5V: now also A1.5V (+5V)
- net BTN1: now also A1.D2
- net BTN2: now also A1.D3
- net BTN3: now also A1.D18 (D18/TX1)
- net GND: now also A1.GND
- net LED_DIN: now also A1.D5
- net MISO: now also A1.D50 (D50/MISO)
- net MOSI: now also A1.D51 (D51/MOSI)
- net RST: now also A1.D9
- net SCK: now also A1.D52 (D52/SCK)
- net SS1: now also A1.D10
- net SS2: now also A1.D8
- net SS3: now also A1.D7
- net SS4: now also A1.D6
- no-connect marks 18 -> 66
Other:
- note added: "Notes: - Power the RC522 from 3.3 V - NOT 5 V! - SPI on the Mega: MISO = D50, MOSI = D51, SCK = D52 (also on the ICSP header). D11-D13 are NOT SPI on the Mega! - SCK/MOSI/MISO and RST are shared by all 4 readers, SDA/SS is individual per reader. - D53 (hardware SS) stays unconnected; SPI.begin() keeps it an output. - The IRQ pin of the readers is not used. - Button 1 (D2) = confirm. Buttons use I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"
- note removed: "Notes: - Power the RC522 from 3.3 V - NOT 5 V! - SCK/MOSI/MISO and RST are shared by all 4 readers, SDA/SS is individual per reader. - The IRQ pin of the readers is not used. - Button 1 (D2) = confirm. Buttons use INPUT_PULLUP, pressed = LOW. - Only D2 and D3 are interrupt pins on the UNO. - Pin assignment of buttons 2/3 (D3/D4) is a suggestion. - At low brightness the matrix can run from the UNO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"
